File: PowerSync/PowerSync.sch (KiCad schematic (older format))
At the start: 39 parts, among them K12VDC1 G5RL-K1A-E, K9VAC1 G5RL-K1A-E, Q1 2N3904, Q2 2N3904, U1 74HCT1G04, U2 74HCT1G32, U3 74HCT74, U4 74HCT2G08

Commit message: Add files via upload
Parts:
- removed D1, D2: 1N4001, Diode_THT:D_DO-41_SOD81_P10.16mm_Horizontal, symbol Diode:1N4001
- removed R3, R4: 8k2, Resistor_SMD:R_0805_2012Metric_Pad1.15x1.40mm_HandSolder, symbol Device:R_Small_US
- removed U1: 74HCT1G04, Package_TO_SOT_SMD:SOT-353_SC-70-5, symbol 74xGxx:74LVC1G04
- removed U3: 74HCT74, Package_SO:TSSOP-14_4.4x5mm_P0.65mm, symbol 74xx:74LS74
- removed U4: 74HCT2G08, Package_SO:TSSOP-8_3x3mm_P0.65mm, symbol 74xGxx:74LVC2G08
- added C1: 220n, Capacitor_SMD:C_0805_2012Metric_Pad1.15x1.40mm_HandSolder, symbol Device:C_Small
- added D1: D_Bridge_+A-A, Diode_THT:Diode_Bridge_15.1x15.1x6.3mm_P10.9mm, symbol Device:D_Bridge_+A-A
- added D4: NSR0530HT1G, Diode_SMD:D_SOD-323_HandSoldering, symbol Diode:1N4001
- added R1: 27k, Resistor_SMD:R_0805_2012Metric_Pad1.15x1.40mm_HandSolder, symbol Device:R_Small_US
- added R2: 33k, Resistor_SMD:R_0805_2012Metric_Pad1.15x1.40mm_HandSolder, symbol Device:R_Small_US
- added R7: 220, Resistor_SMD:R_0805_2012Metric_Pad1.15x1.40mm_HandSolder, symbol Device:R_Small_US
- added U1: LM7805_TO220, Package_TO_SOT_THT:TO-220-3_Vertical, symbol Regulator_Linear:LM7805_TO220
- added U2: 74HCT04, Package_SO:TSSOP-14_4.4x5mm_P0.65mm, symbol 74xx:74LS04
- added U3: 74HCT08, Package_SO:TSSOP-14_4.4x5mm_P0.65mm, symbol 74xx:74LS08
- C2: renamed from C6; value 2u2 -> 1u
- R3: renamed from R1; value 33k -> 22k
- R4: renamed from R2; value 20k -> 10k
- renumbered C9 to C10, C10 to C11, C1 to C4, C2 to C5, C4 to C6, C5 to C7, C7 to C8, C8 to C9, D3 to D2, D4 to D3, U2 to U4
Connections:
- net +12V: now also C1.1, U1.1 (VI)
- net +5V: now also D4.2 (A), R1.1, R7.1; no longer C4.1, C5.1, C6.1, C7.1, C8.1, C9.1, D2.1 (K), D3.1 (K), K12VDC1.9 (SR+), K9VAC1.9 (SR+), U4.5 (VCC)
- net +9VA: now also D1.2 (~~)
- net GND: now also C1.2, D1.3 (-), R2.2, U1.2 (GND), U2.11, U2.13, U2.7 (GND), U3.7 (GND)
- net NEUT: now also D1.4 (~~)
- net at R5.1: now also U2.5, U3.6
- net at R6.1: now also U3.3
- net DET_9VAC: now reaches R3.2, R4.1
- net DET_9VAC: now also U2.9, U3.10, U3.12; no longer C2.1, U4.1
- net at U4.2: now also U3.11; no longer U4.4
- net at C3.1, R3.1: now also D1.1 (+)
- new net: U2.8, U4.1
- new net: U3.2, U4.4
- new net: U2.6, U3.1
- new net: U3.4, U3.8
- new net: U2.4, U3.5
- new net: U2.2, U3.13
- new net DET_5V: R7.2, U2.1, U3.9
- new net TIMER-5V: C2.1, R1.2, R2.1, U2.3
- new net VCC: C4.1, C5.1, C6.1, C7.1, C8.1, C9.1, D2.1 (K), D3.1 (K), D4.1 (K), K12VDC1.9 (SR+), K9VAC1.9 (SR+), U1.3 (VO), U2.14 (VCC), U3.14 (VCC), U4.5 (VCC)
Other:
- note added: "Isolated 5VDC supply so the computer system & drives cannot\ndrain C4 used for reserve power for resetting relay coils."
- moved on the sheet: C2, C3, C4, C5, C6, C7, C8, IN-1, IN-2, IN-3, IN-4, IN-5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
